File: panel/WS_panel/WS_panel.kicad_pcb (KiCad board)
At the start: 2 copper layers, 40.3 x 128.5 mm, 28 parts, among them J1 PJ301M-12, SW1 NKK-Switches

Commit message: updated panel
Parts:
- removed the REF** at (7.00, 111.0)
- removed the REF** at (20.4, 111.0)
- removed the REF** at (34.0, 83.0)
- removed the REF** at (20.4, 97.0)
- removed the REF** at (7.00, 83.0)
- removed the REF** at (54.0, 41.5)
- removed the REF** at (34.0, 111.0)
- removed the REF** at (20.5, 83.0)
- removed the REF** at (7.00, 97.0)
- removed the REF** at (34.0, 97.0)
- added R56: potentiometer, Eurocad:Alpha9mmPot, F.Cu at (112.5, -67.7)
- added R7: potentiometer_plastic_shaft, Eurocad:Plastic_Shaft_Pot_9mm, F.Cu at (-139.1, 54.4)
- added REF**: jack_pot, Eurocad:jack_pot, F.Cu at (59.5, 17.5)
- added REF**: jack_pot, Eurocad:jack_pot, F.Cu at (10.0, 17.5)
- added REF**: jack_pot, Eurocad:jack_pot, F.Cu at (15.0, 33.9)
- added REF**: jack_pot, Eurocad:jack_pot, F.Cu at (39.0, 17.5)
- added REF**: jack_pot, Eurocad:jack_pot, F.Cu at (91.5, 17.5)
- added REF**: mounting_hole, Eurocad:mounting_hole_copy, F.Cu at (124.0, 3.00)
- added REF**: jack_pot, Eurocad:jack_pot, F.Cu at (76.2, 70.6)
- added REF**: jack_pot, Eurocad:jack_pot, F.Cu at (112.5, -48.9)
- added REF**: jack_pot, Eurocad:jack_pot, F.Cu at (117.5, 52.2)
- added REF**: jack_pot, Eurocad:jack_pot, F.Cu at (76.2, 89.0)
- added REF**: jack_pot, Eurocad:jack_pot, F.Cu at (76.2, 52.2)
- added REF**: jack_pot, Eurocad:jack_pot, F.Cu at (35.2, 70.6)
- added REF**: jack_pot, Eurocad:jack_pot, F.Cu at (35.2, 33.9)
- added REF**: jack_pot, Eurocad:jack_pot, F.Cu at (97.2, 33.9)
- added REF**: jack_pot, Eurocad:jack_pot, F.Cu at (97.2, 70.6)
- added REF**: jack_pot, Eurocad:jack_pot, F.Cu at (122.5, 17.5)
- added REF**: jack_pot, Eurocad:jack_pot, F.Cu at (55.8, 89.0)
- added REF**: jack_pot, Eurocad:jack_pot, F.Cu at (97.2, 52.2)
- added REF**: jack_pot, Eurocad:jack_pot, F.Cu at (101.0, 17.5)
- added REF**: jack_pot, Eurocad:jack_pot, F.Cu at (55.8, 70.6)
- added REF**: jack_pot, Eurocad:jack_pot, F.Cu at (19.5, 17.5)
- added REF**: jack_pot, Eurocad:jack_pot, F.Cu at (113.0, 17.5)
- added REF**: jack_pot, Eurocad:jack_pot, F.Cu at (35.2, 89.0)
- added REF**: jack_pot, Eurocad:jack_pot, F.Cu at (117.5, 89.0)
- added REF**: jack_pot, Eurocad:jack_pot, F.Cu at (29.5, 17.5)
- added REF**: jack_pot, Eurocad:jack_pot, F.Cu at (117.5, 70.6)
- added REF**: jack_pot, Eurocad:jack_pot, F.Cu at (76.2, 33.9)
- added REF**: jack_pot, Eurocad:jack_pot, F.Cu at (-65.0, -1.30)
- added REF**: jack_pot, Eurocad:jack_pot, F.Cu at (70.5, 17.5)
- added REF**: jack_pot, Eurocad:jack_pot, F.Cu at (50.0, 17.5)
- added REF**: jack_pot, Eurocad:jack_pot, F.Cu at (35.2, 52.2)
- added REF**: jack_pot, Eurocad:jack_pot, F.Cu at (112.5, -67.7)
- added REF**: jack_pot, Eurocad:jack_pot, F.Cu at (55.8, 33.9)
- added REF**: jack_pot, Eurocad:jack_pot, F.Cu at (117.5, 33.9)
- added REF**: jack_pot, Eurocad:jack_pot, F.Cu at (55.8, 52.2)
- added REF**: jack_pot, Eurocad:jack_pot, F.Cu at (97.2, 89.0)
- added REF**: jack_pot, Eurocad:jack_pot, F.Cu at (80.0, 17.5)
- added SW1: NKK-Switches, scannerFilter:NKK-Switch-1pole, F.Cu at (112.5, -30.4)
- added SW1: NKK-Switches, scannerFilter:NKK-Switch-1pole, F.Cu at (15.4, 61.0)
- added SW1: NKK-Switches, scannerFilter:NKK-Switch-1pole, F.Cu at (15.4, 82.0)
- moved J1 193.1 mm to (-125.5, 97.5), turned to 180 degrees
- moved J1 181.5 mm to (-114.5, 113.0)
- moved J1 181.5 mm to (-101.0, 99.0)
- moved J1 181.5 mm to (-101.0, 85.0)
- moved J1 181.5 mm to (-87.5, 113.0)
- moved J1 181.5 mm to (-87.5, 99.0)
- moved J1 181.5 mm to (-114.5, 99.0)
- moved J1 181.5 mm to (-101.0, 113.0)
- moved SW1 181.5 mm to (-101.5, 63.0)
- moved REF** 166.9 mm to (-136.7, -21.6) (x2)
- moved REF** 166.9 mm to (-119.3, -17.5)
- moved J1 132.2 mm to (112.5, -48.9)
- moved REF** 116.8 mm to (-95.5, 6.50) (x2)
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Other:
- board size 40.3 x 128.5 mm -> 131.5 x 128.5 mm
- board text added: "CV"
- board text added: "CV1"
- board text added: "CVX1"
- board text added: "CVX2"
- board text added: "CVX3"
- board text added: "CVX4"
- board text added: "CVY1"
- board text added: "CVY2"
- board text added: "CVY3"
- board text added: "CVY4"
- board text added: "GATE"
- board text added: "GATE1"
- board text added: "GATE2"
- board text added: "GATE3"
- board text added: "GATE4"
- board text added: "Parts Palette"
- board text added: "Position"
- board text added: "RESET"
- board text added: "T E S S E R A"
- board text added: "TEXT"
- board text added: "pcb safe zones"
- board text removed: "M O N A D"
- board text removed: "NOISE"
- board text removed: "V/OCT"
